File: PcbDesign/TurretCtl/TurretCtl.kicad_pcb (KiCad board)
At the start: 2 copper layers, 27 parts, among them J1 PWR, J2 St1, J3 St2, J4 Sv1, J5 Sense, J6 Sv2, U1 DRV8886, U2 DRV8886

Commit message: TurretCtl revision
Parts:
- moved J2 96.4 mm to (191.7, 136.8)
- moved R2 76.8 mm to (199.5, 116.3), turned to -90 degrees
- moved R1 76.7 mm to (199.5, 114.0), turned to 90 degrees
- moved C6 71.8 mm to (193.7, 109.0)
- moved C7 71.1 mm to (183.8, 103.6), turned to 0 degrees
- moved C5 71.1 mm to (193.9, 121.4)
- moved J3 65.2 mm to (175.2, 136.8)
- moved C11 62.0 mm to (154.2, 109.0), turned to 180 degrees
- moved R3 61.6 mm to (160.4, 116.1), turned to -90 degrees
- moved R4 59.7 mm to (160.4, 113.8)
- moved U1 58.2 mm to (189.4, 115.1), turned to 0 degrees
- moved C4 48.9 mm to (178.9, 109.0), turned to 180 degrees
- moved C12 48.1 mm to (154.7, 121.4), turned to 180 degrees
- moved C1 44.2 mm to (185.0, 109.0), turned to 0 degrees
- moved C2 43.0 mm to (185.0, 121.4), turned to 0 degrees
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Connections:
- U2 pad 19: /Step1 -> /Step2
- U2 pad 20: /Dir1 -> /Dir2
Routing:
- net /Sw-O: track 0.00 -> 102.6 mm
- net /Stepper2/AOUT2: track 5.89 -> 59.1 mm
- net /Stepper2/AOUT1: track 7.93 -> 60.9 mm
- net /Stepper2/BOUT1: track 2.79 -> 54.5 mm
- net /Stepper2/BOUT2: track 4.66 -> 55.0 mm
- net Net-(U2-DVDD): track 0.00 -> 47.6 mm
- net /Sig2: track 0.00 -> 46.6 mm
- net /Sig1: track 0.00 -> 45.7 mm
- net /Step1: track 4.64 -> 45.0 mm
- net /Dir2: track 0.00 -> 31.9 mm, vias 0 -> 1
- net /Dir1: track 4.90 -> 35.0 mm
- net /Stepper1/BOUT1: track 3.16 -> 31.9 mm
- net /Stepper1/AOUT2: track 5.78 -> 34.3 mm
- net /Stepper1/BOUT2: track 4.66 -> 32.4 mm
- net /Step2: track 0.00 -> 27.6 mm, vias 0 -> 1
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Other:
- copper layers 2 -> 4

Commit message: TurretCtl V0.1
Connections:
- U1 pad 25: (no net) -> /GND
- U2 pad 25: (no net) -> /GND
Routing:
- net /Sw-I: track 5.00 -> 83.7 mm
- net /Sig2: track 46.6 -> 81.0 mm
- net /VM: track 65.4 -> 96.0 mm, vias 0 -> 2
- net /Stepper1/AOUT1: track 35.3 -> 39.9 mm
- net /Stepper2/AOUT1: track 60.9 -> 63.0 mm
- net /Stepper1/AOUT2: track 34.3 -> 35.8 mm
- net /GND: track 83.0 -> 84.5 mm
- net /Stepper1/BOUT1: track 31.9 -> 32.4 mm
- added copper zone on B.Cu, net /GND
- added copper zone on In2.Cu, net /VM
Other:
- board outline added: 94 x 104.1 mm
