File: PcbDesign/pump-lights-siren/pump-lights-siren.kicad_sch (KiCad schematic)
At the start: 7 parts, among them Q1 Q_NMOS_GDS, Q2 Q_NMOS_GDS, Q3 Q_NMOS_GDS, Q4 Q_Photo_NPN_CBE, Q5 Q_Photo_NPN_CBE, Q6 Q_Photo_NPN_CBE

Commit message: Mosfet design
Parts:
- removed Q4, Q5, Q6: Q_Photo_NPN_CBE, symbol Device:Q_Photo_NPN_CBE
- added D1, D10, D11, D2, D3, D4, D5, D6, D7, D8, D9: LED_Small, symbol Device:LED_Small
- added J1, J2, J3, J4: Conn_01x02_Socket, symbol Connector:Conn_01x02_Socket
- added R1, R2, R3: 50, symbol Device:R_Small
- added R10, R11, R12, R13, R14, R15, R16, R17, R4, R5, R6, R7, R8, R9: 1k, symbol Device:R_Small
- added T1, T2, T3: ~, symbol opto:V0617A
- Q1, Q2, Q3: footprint (none) -> Package_TO_SOT_THT:TO-220-3_Vertical
Connections:
- net +12V: now also XA1.VIN, D11.2 (A)
- net +12VA: now also Q1.2 (D), Q2.2 (D), Q3.2 (D), D10.2 (A), J4.1 (Pin_1), T1.4 (Collector), T2.4 (Collector), T3.4 (Collector)
- net GND: now also XA1.GND1 (GND), XA1.GND2 (GND), XA1.GND3 (GND), R1.1, R10.2, R11.2, R12.2, R17.2, R2.1, R3.1
- net GNDA: now also D4.1 (K), D5.1 (K), D6.1 (K), J1.2 (Pin_2), J2.2 (Pin_2), J3.2 (Pin_2), J4.2 (Pin_2), R13.2, R14.2, R15.2, R16.2
- net a3: now also D3.2 (A), T3.1 (LogicV)
- net a4: now also D2.2 (A), T2.1 (LogicV)
- net a5: now also D1.2 (A), T1.1 (LogicV)
- net at Q3.1 (G): now also R8.2, R9.1
- net at Q3.3 (S): now also D7.2 (A), J3.1 (Pin_1)
- net at Q1.1 (G): now also R4.2, R5.1
- net at Q1.3 (S): now also D9.2 (A), J1.1 (Pin_1)
- net at Q2.1 (G): now also R6.2, R7.1
- net at Q2.3 (S): now also D8.2 (A), J2.1 (Pin_1)
- net a2: no longer names the net of XA1.A2
- new net: R3.2, T3.2 (LogicGnd)
- new net: R8.1, T3.3 (Emitter)
- new net: D3.1 (K), R12.1
- new net: D7.1 (K), R13.1
- new net: D4.2 (A), R5.2
- new net: D1.1 (K), R10.1
- new net: D11.1 (K), R17.1
- new net: R2.2, T2.2 (LogicGnd)
- new net: R6.1, T2.3 (Emitter)
- new net: R1.2, T1.2 (LogicGnd)
- new net: R4.1, T1.3 (Emitter)
- new net: D6.2 (A), R9.2
- new net: D5.2 (A), R7.2
- new net: D10.1 (K), R16.1
- new net: D8.1 (K), R14.1
- new net: D9.1 (K), R15.1
- new net: D2.1 (K), R11.1
Other:
- moved on the sheet: Q1, XA1

Commit message: V1
Parts:
- removed D5, D6, D8: LED_Small, symbol Device:LED_Small
- removed J2: Conn_01x02_Socket, symbol Connector:Conn_01x02_Socket
- removed R2, R3: 50, symbol Device:R_Small
- removed R6, R7, R8: 1k, symbol Device:R_Small
- added D11, D14: D_Small, Package_TO_SOT_THT:TO-220-2_Horizontal_TabDown, symbol Device:D_Small
- added D12, D13, D9: LED_Small, LED_SMD:LED_0603_1608Metric_Pad1.05x0.95mm_HandSolder, symbol Device:LED_Small
- added J4: Conn_01x02_Socket, Connector_Phoenix_MC:PhoenixContact_MC_1,5_2-G-3.5_1x02_P3.50mm_Horizontal, symbol Connector:Conn_01x02_Socket
- added R11, R15, R16, R17: 1k, Resistor_SMD:R_0603_1608Metric_Pad0.98x0.95mm_HandSolder, symbol Device:R_Small
- added R4: 50, Resistor_SMD:R_0603_1608Metric_Pad0.98x0.95mm_HandSolder, symbol Device:R_Small
- D1: renamed from D11; footprint (none) -> LED_SMD:LED_0603_1608Metric_Pad1.05x0.95mm_HandSolder
- D2: renamed from D10; footprint (none) -> LED_SMD:LED_0603_1608Metric_Pad1.05x0.95mm_HandSolder
- D3: renamed from D1; footprint (none) -> LED_SMD:LED_0603_1608Metric_Pad1.05x0.95mm_HandSolder
- D4: renamed from D2; footprint (none) -> LED_SMD:LED_0603_1608Metric_Pad1.05x0.95mm_HandSolder
- D5: renamed from D3; footprint (none) -> LED_SMD:LED_0603_1608Metric_Pad1.05x0.95mm_HandSolder
- D6: renamed from D4; footprint (none) -> LED_SMD:LED_0603_1608Metric_Pad1.05x0.95mm_HandSolder
- D7: footprint (none) -> LED_SMD:LED_0603_1608Metric_Pad1.05x0.95mm_HandSolder
- D8: renamed from D9; footprint (none) -> LED_SMD:LED_0603_1608Metric_Pad1.05x0.95mm_HandSolder
- J1: renamed from J4; footprint (none) -> Connector_Phoenix_MC:PhoenixContact_MC_1,5_2-G-3.5_1x02_P3.50mm_Horizontal
- J2: renamed from J1; footprint (none) -> Connector_Phoenix_MC:PhoenixContact_MC_1,5_2-G-3.5_1x02_P3.50mm_Horizontal
- J3: footprint (none) -> Connector_Phoenix_MC:PhoenixContact_MC_1,5_2-G-3.5_1x02_P3.50mm_Horizontal
- Q1, Q2, Q3: footprint Package_TO_SOT_THT:TO-220-3_Vertical -> Package_TO_SOT_THT:TO-220-3_Horizontal_TabDown
- R1: renamed from R17; footprint (none) -> Resistor_SMD:R_0603_1608Metric_Pad0.98x0.95mm_HandSolder
- R10: renamed from R5; footprint (none) -> Resistor_SMD:R_0603_1608Metric_Pad0.98x0.95mm_HandSolder
- R12: renamed from R15; footprint (none) -> Resistor_SMD:R_0603_1608Metric_Pad0.98x0.95mm_HandSolder
- R13, R9: footprint (none) -> Resistor_SMD:R_0603_1608Metric_Pad0.98x0.95mm_HandSolder
- R14: value 1k -> 50; footprint (none) -> Resistor_SMD:R_0603_1608Metric_Pad0.98x0.95mm_HandSolder
- R2: renamed from R16; footprint (none) -> Resistor_SMD:R_0603_1608Metric_Pad0.98x0.95mm_HandSolder
- R3: renamed from R1; footprint (none) -> Resistor_SMD:R_0603_1608Metric_Pad0.98x0.95mm_HandSolder
- R5: renamed from R10; footprint (none) -> Resistor_SMD:R_0603_1608Metric_Pad0.98x0.95mm_HandSolder
- R6: renamed from R11; footprint (none) -> Resistor_SMD:R_0603_1608Metric_Pad0.98x0.95mm_HandSolder
- R7: renamed from R12; footprint (none) -> Resistor_SMD:R_0603_1608Metric_Pad0.98x0.95mm_HandSolder
- R8: renamed from R4; footprint (none) -> Resistor_SMD:R_0603_1608Metric_Pad0.98x0.95mm_HandSolder
- T1, T2, T3: footprint (none) -> Package_DIP:DIP-4_W7.62mm
Connections:
- net +12V: now also D8.2 (A), J2.1 (Pin_1), T1.4 (Collector), T3.4 (Collector), D13.2 (A), D14.1 (K), J4.1 (Pin_1)
- net GND: now also Q1.3 (S), Q3.3 (S), R10.2, R14.1, R16.2, R4.1
- net a3: now also T2.1 (LogicV); no longer T3.1 (LogicV)
- net a4: now also T3.1 (LogicV); no longer T2.1 (LogicV)
- net at T3.2 (LogicGnd): now also R14.2
- net at T3.3 (Emitter): now also R15.1
- net at R13.1: now also D9.1 (K); no longer D7.1 (K)
- net at D6.2 (A): now also Q1.1 (G), R8.2; no longer R10.2
- net at T2.2 (LogicGnd): now also R4.2
- net at T2.3 (Emitter): now also R9.1
- net at Q3.1 (G): now also D12.2 (A), R15.2; no longer R9.1
- net GNDPWR: now reaches Q2.3 (S)
- net GNDPWR: now also J1.2 (Pin_2), R2.2, R11.2
- net at R9.2: now also D7.2 (A), Q2.1 (G)
- removed net +12VA: D2.2 (A), J1.1 (Pin_1), Q1.2 (D), Q2.2 (D), Q3.2 (D), T1.4 (Collector), T2.4 (Collector), T3.4 (Collector)
- removed net GNDA: D6.1 (K), J1.2 (Pin_2), J2.2 (Pin_2), J3.2 (Pin_2), R12.2, R13.2, R14.2, R2.2
- new net: D14.2 (A), J4.2 (Pin_2), Q3.2 (D), R17.2
- new net: D12.1 (K), R16.1
- new net: D6.1 (K), R10.1
- new net: D7.1 (K), R11.1
- new net: D11.2 (A), J3.2 (Pin_2), Q2.2 (D), R13.2
- new net: J2.2 (Pin_2), Q1.2 (D), R12.2
- new net: D13.1 (K), R17.1
- new net +12P: D11.1 (K), D2.2 (A), D9.2 (A), J1.1 (Pin_1), J3.1 (Pin_1), T2.4 (Collector)
- no-connect marks 0 -> 30
Other:
- note added: "Lights"
- note added: "Pump"
- note added: "Siren"
- moved on the sheet: D6, D8, J2, R10, R12, R8
